File: MFD.kicad_sch (KiCad schematic)
At the start: 39 parts, among them U1 4051, U2 ProMicro

Commit message: Adds mounting holes to schematic\nReroutes some tracks
Parts:
- added H1, H2, H3, H4: MountingHole, MountingHole:MountingHole_5.3mm_M5, symbol Mechanical:MountingHole

Commit message: re-adds open hardware silkscreen adds open hardware symbol to schematic adds net names
Parts:
- added SYM1: Logo_Open_Hardware_Small, Symbol:OSHW-Logo2_7.3x6mm_SilkScreen, symbol Graphic:Logo_Open_Hardware_Small
Connections:
- net COL_3: now reaches SW_L3.1, SW_M/B1.1, SW_T5.1, SW_TSD1.1, U1.12 (X3)
- net ROW_C: now reaches SW_B5.2, SW_B6.2, SW_L1.2, SW_L2.2, SW_L3.2, SW_L4.2, SW_L5.2, SW_L6.2, U2.7 (D4/A6)
- net COL_6: now reaches SW_B6.1, SW_R4.1, SW_T2.1, SW_VID1.1, U1.2 (X6)
- net ROW_B: now reaches SW_B2.2, SW_B3.2, SW_B4.2, SW_M/B1.2, SW_R3.2, SW_R4.2, SW_R5.2, SW_R6.2, U2.6 (SCL/D3)
- net COL_7: now reaches SW_B5.1, SW_Fav1.1, SW_R3.1, SW_T1.1, U1.4 (X7)
- net ROW_D: now reaches SW_AC1.2, SW_COM1.2, SW_FCR1.2, SW_Fav1.2, SW_TSD1.2, SW_VID1.2, SW_WPN1.2, U2.8 (D5)
- net COL_1: now reaches SW_B3.1, SW_FCR1.1, SW_L5.1, SW_R1.1, U1.14 (X1)
- net COL_5: now reaches SW_COM1.1, SW_L1.1, SW_R5.1, SW_T3.1, U1.5 (X5)
- net ROW_A: now reaches SW_R1.2, SW_R2.2, SW_T1.2, SW_T2.2, SW_T3.2, SW_T4.2, SW_T5.2, SW_T6.2, U2.5 (SDA/D2)
- net COL_2: now reaches SW_B2.1, SW_L4.1, SW_T6.1, SW_WPN1.1, U1.15 (X2)
- net COL_4: now reaches SW_AC1.1, SW_L2.1, SW_R6.1, SW_T4.1, U1.1 (X4)
- net MUX_Common: now reaches R3.2, U1.3 (X), U2.13 (D10)
- net ADDR_1: now reaches U1.10 (B), U2.11 (D8/A8)
- net ADDR_0: now reaches U1.11 (A), U2.12 (D9/A9)
- net COL_0: now reaches SW_B4.1, SW_L6.1, SW_R2.1, U1.13 (X0)
- net MUX_Inhibbit: now reaches U1.6 (Inh), U2.9 (D6/A7)
- net ADDR_2: now reaches U1.9 (C), U2.10 (D7)
- net at RV_BRT1.2: now also R2.2; no longer R1.2
- net Analog_VID: now reaches R2.1, U2.17 (A0)
- net Analog_BRT: now reaches R1.1, U2.18 (A1)
- net at RV_VID1.2: now also R1.2; no longer R2.2
Other:
- moved on the sheet: RV_BRT1, RV_VID1
